File: stardust-shield/stardust.sch (KiCad schematic (older format))
At the start: 13 parts, among them J1 BEXUS 28V, J2 Pololu J8557, J3 Pololu J9251, J4 DS3231M, U1 MCP1416, U3 MCP1416, U5 DS18B20, U6 DS18B20, U8 DHT22, U9 SSCDRNN015PASA5

Commit message: main pcb
Parts:
- removed U1, U3: MCP1416, Package_TO_SOT_SMD:SOT-23-5, symbol Driver_FET:MCP1416
- added U1, U2: IRFL210, Package_TO_SOT_SMD:SOT-223-3_TabPin2, symbol Regulator_Linear:LM337_SOT223
Connections:
- net labels added: 1Wire-1, 1Wire-2, 1Wire-3, SPI-SS-Pressure-1, SPI-SS-Pressure-2
- net labels removed: 1Wire, SPI, SPI-SS-Pressure, VCC
- wire segments 38 -> 44
Other:
- moved on the sheet: DSUB-1, DSUB-2, J1, J2, J3, J4, U5, U6, U8, XA1

Commit message: add footprints, clear board
Parts:
- removed U1, U2: IRFL210, Package_TO_SOT_SMD:SOT-223-3_TabPin2, symbol Regulator_Linear:LM337_SOT223
- removed U9: SSCDRNN015PASA5, Package_DIP:DIP-8_W8.89mm_SMDSocket_LongPads, symbol Sensor_Pressure:MS5607-02BA
- added U1, U2: IRFL210, Package_TO_SOT_SMD:SOT-223, symbol irfl210:IRFL210
- added U9: SSCDRNN015PASA5, Package_DIP:DIP-8_W8.89mm_SMDSocket_LongPads, symbol sscdrnn015pasa5:SSCDRNN015PASA5
Connections:
- wire segments 44 -> 48
Other:
- moved on the sheet: DSUB-1, DSUB-2, J1, J2, J3, J4, U5, U6, U8, XA1

Commit message: move mosfet to mech board, controll pump via gnd
Parts:
- removed U1, U2: IRFL210, Package_TO_SOT_SMD:SOT-223, symbol irfl210:IRFL210
Connections:
- net labels added: Pump-GPIO
- net labels removed: Pump-1, Pump-2, Pump-GPIO-1, Pump-GPIO-2
Changed lines of the file:
@@
 	1    0    0    -1
 $EndComp
-$Comp
-L power:+5V #PWR0105
-U 1 1 5EB55AC0
-P 8450 2750
-F 0 "#PWR0105" H 8450 2600 50  0001 C CNN
-F 1 "+5V" H 8465 2923 50  0000 C CNN
-F 2 "" H 8450 2750 50  0001 C CNN
-F 3 "" H 8450 2750 50  0001 C CNN
-	1    8450 2750
-	-1   0    0    -1
-$EndComp
-Text GLabel 8650 3050 0    50   Input ~ 0
-Pump-1
 Wire Wire Line
 	8450 2950 8450 2750
@@
 Wire Wire Line
 	8650 3750 8450 3750
-Text GLabel 8650 3650 0    50   Input ~ 0
-Pump-2
 $Comp
 L Connector:DB9_Male_MountingHoles DSUB-1
@@
 Text GLabel 9300 12500 2    50   Input ~ 0
 SPI-MOSI
-Text GLabel 9300 9900 2    50   Input ~ 0
-Pump-GPIO-1
 Text GLabel 9300 9700 2    50   Input ~ 0
-Pump-GPIO-2
-Text GLabel 4800 12750 2    50   Input ~ 0
-Pump-2
+Pump-GPIO
 $Comp
 L power:+5V #PWR0134
@@
 	1    0    0    -1
 $EndComp
-Text GLabel 2850 12750 2    50   Input ~ 0
-Pump-1
 Text GLabel 9300 11500 2    50   Input ~ 0
 SPI-SS-Pressure-1
@@
 Connection ~ 6500 11900
 $Comp
-L irfl210:IRFL210 U2
-U 1 1 5EA5E9FB
-P 4500 13050
-F 0 "U2" H 4500 13227 50  0000 C CNN
-F 1 "IRFL210" H 4500 13136 50  0000 C CNN
-F 2 "Package_TO_SOT_SMD:SOT-223" H 4500 13200 50  0001 C CNN
-F 3 "https://sensing.honeywell.com/index.php?ci_id=151134" H 4500 13000 50  0001 C CNN
-	1    4500 13050
-	1    0    0    -1
-$EndComp
-$Comp
-L irfl210:IRFL210 U1
-U 1 1 5EA60E65
-P 2550 13050
-F 0 "U1" H 2550 13227 50  0000 C CNN
-F 1 "IRFL210" H 2550 13136 50  0000 C CNN
-F 2 "Package_TO_SOT_SMD:SOT-223" H 2550 13200 50  0001 C CNN
-F 3 "https://sensing.honeywell.com/index.php?ci_id=151134" H 2550 13000 50  0001 C CNN
-	1    2550 13050
-	1    0    0    -1
-$EndComp
-$Comp
-L power:+12V #PWR0108
-U 1 1 5EC6A2FB
-P 2150 12650
-F 0 "#PWR0108" H 2150 12500 50  0001 C CNN
-F 1 "+12V" H 2165 12823 50  0000 C CNN
-F 2 "" H 2150 12650 50  0001 C CNN
-F 3 "" H 2150 12650 50  0001 C CNN
-	1    2150 12650
-	1    0    0    -1
-$EndComp
-Text GLabel 2550 12450 1    50   Input ~ 0
-Pump-GPIO-1
-Text GLabel 4500 12450 1    50   Input ~ 0
-Pump-GPIO-2
-$Comp
-L power:+12V #PWR0110
-U 1 1 5EC7A67C
-P 4100 12650
-F 0 "#PWR0110" H 4100 12500 50  0001 C CNN
-F 1 "+12V" H 4115 12823 50  0000 C CNN
-F 2 "" H 4100 12650 50  0001 C CNN
-F 3 "" H 4100 12650 50  0001 C CNN
-	1    4100 12650
-	1    0    0    -1
-$EndComp
-Wire Wire Line
-	4100 12650 4100 12750
-Wire Wire Line
-	4100 12750 4200 12750
-$Comp
 L sscdrnn015pasa5:SSCDRNN015PASA5 U9
 U 1 1 5EA83F3B
@@
 $EndComp
 Wire Wire Line
-	2250 12750 2150 12750
-Wire Wire Line
-	2150 12750 2150 12650
+	8050 3650 8050 2750
+Wire Wire Line
+	8050 3650 8650 3650
+Wire Wire Line
+	8250 3050 8250 2750
+Wire Wire Line
+	8250 3050 8650 3050
+$Comp
+L power:+5V #PWR?
+U 1 1 5EA555FA
+P 8450 2750
+F 0 "#PWR?" H 8450 2600 50  0001 C CNN
+F 1 "+5V" H 8465 2923 50  0000 C CNN
+F 2 "" H 8450 2750 50  0001 C CNN
+F 3 "" H 8450 2750 50  0001 C CNN
+	1    8450 2750
+	1    0    0    -1
+$EndComp
+$Comp
+L power:+12V #PWR?
+U 1 1 5EA5592B
+P 8250 2750
+F 0 "#PWR?" H 8250 2600 50  0001 C CNN
+F 1 "+12V" H 8265 2923 50  0000 C CNN
+F 2 "" H 8250 2750 50  0001 C CNN
+F 3 "" H 8250 2750 50  0001 C CNN
+	1    8250 2750
+	1    0    0    -1
+$EndComp
+$Comp
+L power:+12V #PWR?
+U 1 1 5EA55CD7
+P 8050 2750
+F 0 "#PWR?" H 8050 2600 50  0001 C CNN
+F 1 "+12V" H 8065 2923 50  0000 C CNN
+F 2 "" H 8050 2750 50  0001 C CNN
+F 3 "" H 8050 2750 50  0001 C CNN
+	1    8050 2750
+	1    0    0    -1
+$EndComp
+Text GLabel 8650 3350 0    50   Input ~ 0
+Pump-GPIO
 $EndSCHEMATC

Commit message: add pump pull-down, clean up paths
Parts:
- added R1: 10k, Resistor_SMD:R_0603_1608Metric, symbol Device:R
Connections:
- net DHT22-1: now also XA1.D27; no longer XA1.D29
- net DHT22-2: now also XA1.D41; no longer XA1.D39
- net GND: now also R1.2
- net Pump-GPIO: now also XA1.D29, R1.1; no longer XA1.D23
- net SPI-SS-Pressure-1: now also XA1.D39; no longer XA1.D41
- net SPI-SS-Pressure-2: now also XA1.D25; no longer XA1.D27
Changed lines of the file:
@@
 Text GLabel 8650 3250 0    50   Input ~ 0
 I2C-SCL
-Wire Wire Line
-	8950 4150 8950 3950
 $Comp
 L power:GND #PWR0104
 U 1 1 5EB55ABA
-P 8950 4150
-F 0 "#PWR0104" H 8950 3900 50  0001 C CNN
-F 1 "GND" H 8955 3977 50  0000 C CNN
-F 2 "" H 8950 4150 50  0001 C CNN
-F 3 "" H 8950 4150 50  0001 C CNN
-	1    8950 4150
+P 8950 3950
+F 0 "#PWR0104" H 8950 3700 50  0001 C CNN
+F 1 "GND" H 8955 3777 50  0000 C CNN
+F 2 "" H 8950 3950 50  0001 C CNN
+F 3 "" H 8950 3950 50  0001 C CNN
+	1    8950 3950
 	1    0    0    -1
 $EndComp
@@
 	8650 3750 8450 3750
 $Comp
-L Connector:DB9_Male_MountingHoles DSUB-1
-U 1 1 5EBA0FF7
-P 8950 3350
-F 0 "DSUB-1" H 9130 3352 50  0000 L CNN
-F 1 "DB9_Male_MountingHoles" H 9130 3261 50  0000 L CNN
-F 2 "Connector_Dsub:DSUB-9_Male_Horizontal_P2.77x2.84mm_EdgePinOffset4.94mm_Housed_MountingHolesOffset7.48mm" H 8950 3350 50  0001 C CNN
-F 3 " ~" H 8950 3350 50  0001 C CNN
-	1    8950 3350
-	1    0    0    -1
-$EndComp
-$Comp
 L Connector:DB9_Male_MountingHoles DSUB-2
 U 1 1 5EBC672B
@@
 Text GLabel 6700 9300 0    50   Input ~ 0
 I2C-SCL
-Text GLabel 9300 10300 2    50   Input ~ 0
+Text GLabel 9300 10100 2    50   Input ~ 0
 DHT22-1
-Text GLabel 9300 11300 2    50   Input ~ 0
-DHT22-2
-Text GLabel 9300 10100 2    50   Input ~ 0
+Text GLabel 9300 9900 2    50   Input ~ 0
 SPI-SS-Pressure-2
 Text GLabel 9300 10700 2    50   Input ~ 0
@@
 Text GLabel 9300 12500 2    50   Input ~ 0
 SPI-MOSI
-Text GLabel 9300 9700 2    50   Input ~ 0
-Pump-GPIO
 $Comp
 L power:+5V #PWR0134
@@
 	1    0    0    -1
 $EndComp
-Text GLabel 9300 11500 2    50   Input ~ 0
+Text GLabel 9300 11300 2    50   Input ~ 0
 SPI-SS-Pressure-1
 Text GLabel 9300 11100 2    50   Input ~ 0
@@
 Wire Wire Line
 	8250 3050 8250 2750
-Wire Wire Line
-	8250 3050 8650 3050
-$Comp
-L power:+5V #PWR?
+$Comp
+L power:+5V #PWR0105
 U 1 1 5EA555FA
 P 8450 2750
-F 0 "#PWR?" H 8450 2600 50  0001 C CNN
+F 0 "#PWR0105" H 8450 2600 50  0001 C CNN
 F 1 "+5V" H 8465 2923 50  0000 C CNN
 F 2 "" H 8450 2750 50  0001 C CNN
@@
 $EndComp
 $Comp
-L power:+12V #PWR?
+L power:+12V #PWR0108
 U 1 1 5EA5592B
 P 8250 2750
-F 0 "#PWR?" H 8250 2600 50  0001 C CNN
+F 0 "#PWR0108" H 8250 2600 50  0001 C CNN
 F 1 "+12V" H 8265 2923 50  0000 C CNN
 F 2 "" H 8250 2750 50  0001 C CNN
@@
 $EndComp
 $Comp
-L power:+12V #PWR?
+L power:+12V #PWR0109
 U 1 1 5EA55CD7
 P 8050 2750
-F 0 "#PWR?" H 8050 2600 50  0001 C CNN
+F 0 "#PWR0109" H 8050 2600 50  0001 C CNN
 F 1 "+12V" H 8065 2923 50  0000 C CNN
 F 2 "" H 8050 2750 50  0001 C CNN
@@
 	1    0    0    -1
 $EndComp
-Text GLabel 8650 3350 0    50   Input ~ 0
+Text GLabel 7750 3350 0    50   Input ~ 0
 Pump-GPIO
+Text GLabel 9300 10300 2    50   Input ~ 0
+Pump-GPIO
+Wire Wire Line
+	7900 3950 7900 3800
+$Comp
+L power:GND #PWR0110
+U 1 1 5EA88781
+P 7900 3950
+F 0 "#PWR0110" H 7900 3700 50  0001 C CNN
+F 1 "GND" H 7905 3777 50  0000 C CNN
+F 2 "" H 7900 3950 50  0001 C CNN
+F 3 "" H 7900 3950 50  0001 C CNN
+	1    7900 3950
+	-1   0    0    -1
+$EndComp
+Wire Wire Line
+	8250 3050 8650 3050
+$Comp
+L Connector:DB9_Male_MountingHoles DSUB-1
+U 1 1 5EBA0FF7
+P 8950 3350
+F 0 "DSUB-1" H 9130 3352 50  0000 L CNN
+F 1 "DB9_Male_MountingHoles" H 9130 3261 50  0000 L CNN
+F 2 "Connector_Dsub:DSUB-9_Male_Horizontal_P2.77x2.84mm_EdgePinOffset4.94mm_Housed_MountingHolesOffset7.48mm" H 8950 3350 50  0001 C CNN
+F 3 " ~" H 8950 3350 50  0001 C CNN
+	1    8950 3350
+	1    0    0    -1
+$EndComp
+$Comp
+L Device:R R1
+U 1 1 5EA96850
+P 7900 3650
+F 0 "R1" H 7650 3700 50  0000 L CNN
+F 1 "10k" H 7650 3600 50  0000 L CNN
+F 2 "Resistor_SMD:R_0603_1608Metric" V 7830 3650 50  0001 C CNN
+F 3 "~" H 7900 3650 50  0001 C CNN
+	1    7900 3650
+	1    0    0    -1
+$EndComp
+Wire Wire Line
+	7750 3350 7900 3350
+Wire Wire Line
+	7900 3500 7900 3350
+Connection ~ 7900 3350
+Wire Wire Line
+	7900 3350 8650 3350
+Text GLabel 9300 11500 2    50   Input ~ 0
+DHT22-2
 $EndSCHEMATC

Commit message: add db9 models, and update footprints
Parts:
- DSUB-1, DSUB-2: footprint Connector_Dsub:DSUB-9_Male_Horizontal_P2.77x2.84mm_EdgePinOffset4.94mm_Housed_MountingHolesOffset7.48mm -> Connector_Dsub:DSUB-9_Male_Horizontal_P2.77x2.84mm_EdgePinOffset7.70mm_Housed_MountingHolesOffset9.12mm
Changed lines of the file:
@@
 encoding utf-8
 Sheet 1 1
-Title "Stardust Overview"
+Title "Stardust Main PCB"
 Date "17 March 2020"
 Rev "2020/3/14"
@@
 F 0 "DSUB-2" H 9130 5702 50  0000 L CNN
 F 1 "DB9_Male_MountingHoles" H 9130 5611 50  0000 L CNN
-F 2 "Connector_Dsub:DSUB-9_Male_Horizontal_P2.77x2.84mm_EdgePinOffset4.94mm_Housed_MountingHolesOffset7.48mm" H 8950 5700 50  0001 C CNN
+F 2 "Connector_Dsub:DSUB-9_Male_Horizontal_P2.77x2.84mm_EdgePinOffset7.70mm_Housed_MountingHolesOffset9.12mm" H 8950 5700 50  0001 C CNN
 F 3 " ~" H 8950 5700 50  0001 C CNN
 	1    8950 5700
@@
 F 0 "DSUB-1" H 9130 3352 50  0000 L CNN
 F 1 "DB9_Male_MountingHoles" H 9130 3261 50  0000 L CNN
-F 2 "Connector_Dsub:DSUB-9_Male_Horizontal_P2.77x2.84mm_EdgePinOffset4.94mm_Housed_MountingHolesOffset7.48mm" H 8950 3350 50  0001 C CNN
+F 2 "Connector_Dsub:DSUB-9_Male_Horizontal_P2.77x2.84mm_EdgePinOffset7.70mm_Housed_MountingHolesOffset9.12mm" H 8950 3350 50  0001 C CNN
 F 3 " ~" H 8950 3350 50  0001 C CNN
 	1    8950 3350

Commit message: rev.2 init
Parts:
- added J4: Pololu J9251 Servo, Connector_PinSocket_2.54mm:PinSocket_1x05_P2.54mm_Vertical, symbol Connector:Conn_01x05_Female
- renumbered J4 to J5
Connections:
- net +28V: now also J4.3 (Pin_3)
- net +5V: now also J4.1 (Pin_1)
- net GND: now also J4.2 (Pin_2)
Other:
- moved on the sheet: J5
Changed lines of the file:
@@
 $EndDescr
 Wire Wire Line
-	6350 4350 6650 4350
+	6650 4400 6950 4400
 Text GLabel 4800 8500 2    50   Input ~ 0
 1Wire-3
@@
 Text GLabel 4800 9700 2    50   Input ~ 0
 DHT22-3
-Text GLabel 6650 4350 2    50   Input ~ 0
+Text GLabel 6950 4400 2    50   Input ~ 0
 I2C-SDA
 $Comp
@@
 L power:+5V #PWR0134
 U 1 1 5ED92911
-P 6500 4050
-F 0 "#PWR0134" H 6500 3900 50  0001 C CNN
-F 1 "+5V" H 6515 4223 50  0000 C CNN
-F 2 "" H 6500 4050 50  0001 C CNN
-F 3 "" H 6500 4050 50  0001 C CNN
-	1    6500 4050
-	1    0    0    -1
-$EndComp
-$Comp
-L power:GND #PWR0124
-U 1 1 5E955680
-P 6500 4800
-F 0 "#PWR0124" H 6500 4550 50  0001 C CNN
-F 1 "GND" H 6505 4627 50  0000 C CNN
-F 2 "" H 6500 4800 50  0001 C CNN
-F 3 "" H 6500 4800 50  0001 C CNN
-	1    6500 4800
-	-1   0    0    -1
-$EndComp
-$Comp
-L Connector:Conn_01x05_Male J4
+P 6800 4000
+F 0 "#PWR0134" H 6800 3850 50  0001 C CNN
+F 1 "+5V" H 6815 4173 50  0000 C CNN
+F 2 "" H 6800 4000 50  0001 C CNN
+F 3 "" H 6800 4000 50  0001 C CNN
+	1    6800 4000
+	1    0    0    -1
+$EndComp
+$Comp
+L Connector:Conn_01x05_Male J5
 U 1 1 5EC929B6
-P 6150 4450
-F 0 "J4" H 6050 4450 50  0000 C CNN
-F 1 "DS3231M" H 6150 3900 50  0000 C CNN
-F 2 "Connector_PinHeader_2.54mm:PinHeader_1x05_P2.54mm_Vertical" H 6150 4450 50  0001 C CNN
-F 3 "~" H 6150 4450 50  0001 C CNN
-	1    6150 4450
-	1    0    0    -1
-$EndComp
-Wire Wire Line
-	6500 4800 6500 4650
-Wire Wire Line
-	6500 4650 6350 4650
-Wire Wire Line
-	6350 4250 6500 4250
-Wire Wire Line
-	6500 4250 6500 4050
-Text GLabel 6650 4450 2    50   Input ~ 0
+P 6450 4500
+F 0 "J5" H 6350 4500 50  0000 C CNN
+F 1 "DS3231M" H 6450 3950 50  0000 C CNN
+F 2 "Connector_PinHeader_2.54mm:PinHeader_1x05_P2.54mm_Vertical" H 6450 4500 50  0001 C CNN
+F 3 "~" H 6450 4500 50  0001 C CNN
+	1    6450 4500
+	1    0    0    -1
+$EndComp
+Wire Wire Line
+	6800 4700 6650 4700
+Wire Wire Line
+	6650 4300 6800 4300
+Text GLabel 6950 4500 2    50   Input ~ 0
 I2C-SCL
 Wire Wire Line
-	6350 4450 6650 4450
+	6650 4500 6950 4500
 Wire Wire Line
 	5100 4300 4900 4300
@@
 Text GLabel 9300 11500 2    50   Input ~ 0
 DHT22-2
+$Comp
+L power:+5V #PWR?
+U 1 1 5F1ECFCA
+P 5650 4050
+F 0 "#PWR?" H 5650 3900 50  0001 C CNN
+F 1 "+5V" H 5700 4250 50  0000 C CNN
+F 2 "" H 5650 4050 50  0001 C CNN
+F 3 "" H 5650 4050 50  0001 C CNN
+	1    5650 4050
+	1    0    0    -1
+$EndComp
+Wire Wire Line
+	5850 4300 5650 4300
+Wire Wire Line
+	5650 4300 5650 4050
+$Comp
+L power:GND #PWR?
+U 1 1 5F1ECFD2
+P 5650 4650
+F 0 "#PWR?" H 5650 4400 50  0001 C CNN
+F 1 "GND" H 5655 4477 50  0000 C CNN
+F 2 "" H 5650 4650 50  0001 C CNN
+F 3 "" H 5650 4650 50  0001 C CNN
+	1    5650 4650
+	1    0    0    -1
+$EndComp
+Wire Wire Line
+	5650 4650 5650 4400
+Wire Wire Line
+	5650 4400 5850 4400
+$Comp
+L Connector:Conn_01x05_Female J4
+U 1 1 5F1ECFDA
+P 6050 4500
+F 0 "J4" H 6078 4526 50  0000 L CNN
+F 1 "Pololu J9251 Servo" H 5450 4000 50  0000 L CNN
+F 2 "Connector_PinSocket_2.54mm:PinSocket_1x05_P2.54mm_Vertical" H 6050 4500 50  0001 C CNN
+F 3 "~" H 6050 4500 50  0001 C CNN
+	1    6050 4500
+	1    0    0    -1
+$EndComp
+Wire Wire Line
+	5850 4500 5500 4500
+Wire Wire Line
+	5500 4500 5500 4050
+$Comp
+L power:+28V #PWR?
+U 1 1 5F1ECFE2
+P 5500 4050
+F 0 "#PWR?" H 5500 3900 50  0001 C CNN
+F 1 "+28V" H 5450 4250 50  0000 C CNN
+F 2 "" H 5750 4100 50  0001 C CNN
+F 3 "" H 5750 4100 50  0001 C CNN
+	1    5500 4050
+	1    0    0    -1
+$EndComp
+Wire Wire Line
+	6800 4000 6800 4300
+Wire Wire Line
+	6800 4850 6800 4700
+$Comp
+L power:GND #PWR0124
+U 1 1 5E955680
+P 6800 4850
+F 0 "#PWR0124" H 6800 4600 50  0001 C CNN
+F 1 "GND" H 6805 4677 50  0000 C CNN
+F 2 "" H 6800 4850 50  0001 C CNN
+F 3 "" H 6800 4850 50  0001 C CNN
+	1    6800 4850
+	-1   0    0    -1
+$EndComp
 $EndSCHEMATC

Commit message: 2.0
Parts:
- removed J2: Pololu J8557, Connector_PinSocket_2.54mm:PinSocket_1x05_P2.54mm_Vertical, symbol Connector:Conn_01x05_Female
- added J2, J3: Pololu J8557, Connector_PinSocket_2.54mm:PinSocket_1x05_P2.54mm_Vertical, symbol stardust-rescue:Conn_01x05_Female-Connector
- added J7: VMA430, Connector_PinHeader_2.54mm:PinHeader_1x05_P2.54mm_Vertical, symbol stardust-rescue:Conn_01x05_Male-Connector
- added R2, R3, R4: 4.7k, Resistor_SMD:R_0603_1608Metric, symbol Device:R
- added R5, R6, R7, R9: 200m, Resistor_SMD:R_0603_1608Metric, symbol Device:R
- added U1, U2, U3, U4: INA181, Package_TO_SOT_SMD:SOT-23-6, symbol Amplifier_Current:INA181
- DSUB-Sensor1: renamed from DSUB-2; symbol Connector:DB9_Male_MountingHoles -> stardust-rescue:DB9_Male_MountingHoles-Connector
- DSUB-Servo1: renamed from DSUB-1; symbol Connector:DB9_Male_MountingHoles -> stardust-rescue:DB9_Male_MountingHoles-Connector
- J1: symbol Connector_Generic:Conn_01x02 -> stardust-rescue:Conn_01x02-Connector_Generic
- J4: renamed from J3; symbol Connector:Conn_01x05_Female -> stardust-rescue:Conn_01x05_Female-Connector
- J5: renamed from J4; symbol Connector:Conn_01x05_Female -> stardust-rescue:Conn_01x05_Female-Connector
- J6: renamed from J5; symbol Connector:Conn_01x05_Male -> stardust-rescue:Conn_01x05_Male-Connector
- R1: symbol Device:R -> stardust-rescue:R-Device
- U5, U6: symbol Sensor_Temperature:DS18B20 -> stardust-rescue:DS18B20-Sensor_Temperature
- U8: symbol Sensor:DHT11 -> stardust-rescue:DHT11-Sensor
- XA1: symbol Arduino:Arduino_Mega2560_Shield -> stardust-rescue:Arduino_Mega2560_Shield-Arduino
Connections:
- net +12V: now also R7.2, U3.4 (-); no longer DSUB-Servo1.9
- net +28V: now also J1.2 (Pin_2), J2.3 (Pin_3), J3.3 (Pin_3); no longer J1.1 (Pin_1)
- net +5V: now also J7.5 (Pin_5), R2.1, R3.1, R4.1, R5.2, U1.4 (-), U1.6 (V+), U2.6 (V+), U3.6 (V+), U4.6 (V+); no longer DSUB-Servo1.5, J4.1 (Pin_1), J5.1 (Pin_1)
- net 1Wire-1: now also R2.2
- net 1Wire-2: now also R3.2
- net 1Wire-3: now also R4.2
- net GND: now also J1.1 (Pin_1), J2.2 (Pin_2), J3.2 (Pin_2), J7.4 (Pin_4), U1.2 (GND), U1.5 (REF), U2.2 (GND), U2.5 (REF), U3.2 (GND), U3.5 (REF), U4.2 (GND), U4.5 (REF); no longer J1.2 (Pin_2)
- net INA1: now reaches XA1.A1
- net INA1: now also U1.1
- net INA2: now reaches XA1.A2
- net INA2: now also U2.1
- net INA3: now reaches XA1.A3
- net INA3: now also U3.1
- net INA4: now reaches XA1.A4
- net INA4: now also U4.1
- net TX3: now reaches XA1.D14 (D14_TX3)
- net TX3: now also J7.2 (Pin_2)
- net RX3: now reaches XA1.D15 (D15_RX3)
- net RX3: now also J7.3 (Pin_3)
- net TX2: now reaches XA1.D16 (D16_TX2)
- net RX2: now reaches XA1.D17 (D17_RX2)
- net TX1: now reaches XA1.D18 (D18_TX1)
- net RX1: now reaches XA1.D19 (D19_RX1)
- new net: J4.1 (Pin_1), R5.1, U1.3 (+)
- new net: J5.1 (Pin_1), R6.1, U2.3 (+)
- new net: J3.1 (Pin_1), R9.1, U4.3 (+)
- new net: J2.1 (Pin_1), R7.1, U3.3 (+)
- new net +12P: DSUB-Servo1.9, R9.2, U4.4 (-)
- new net +5P: DSUB-Servo1.5, R6.2, U2.4 (-)
Other:
- moved on the sheet: J1, J4, J5, J6

Commit message: final 2.0
Parts:
- removed R1: 10k, Resistor_SMD:R_0603_1608Metric, symbol stardust-rescue:R-Device
- added C1, C2, C3, C4: 1mF, Capacitor_SMD:C_0603_1608Metric_Pad1.05x0.95mm_HandSolder, symbol Device:C
- added D1, D2, D3, D4, D5, D6: LED, LED_SMD:LED_0603_1608Metric_Pad1.05x0.95mm_HandSolder, symbol Device:LED
- added J7'1: VMA430, Connector_PinHeader_2.54mm:PinHeader_1x05_P2.54mm_Vertical, symbol stardust-rescue:Conn_01x05_Male-Connector
- added R12, R13: 10k, Resistor_SMD:R_0603_1608Metric_Pad1.05x0.95mm_HandSolder, symbol Device:R
- added R14, R15, R16, R17, R18, R19: 1k, Resistor_SMD:R_0603_1608Metric_Pad1.05x0.95mm_HandSolder, symbol Device:R
- added R2, R4, R6, R8: 16k, Resistor_SMD:R_0603_1608Metric_Pad1.05x0.95mm_HandSolder, symbol Device:R
- added SW1, SW2: SW_Push, Button_Switch_THT:SW_TH_Tactile_Omron_B3F-10xx, symbol Switch:SW_Push
- R1: renamed from R5; footprint Resistor_SMD:R_0603_1608Metric -> Resistor_SMD:R_0603_1608Metric_Pad1.05x0.95mm_HandSolder
- R10: renamed from R3; footprint Resistor_SMD:R_0603_1608Metric -> Resistor_SMD:R_0603_1608Metric_Pad1.05x0.95mm_HandSolder
- R11: renamed from R4; footprint Resistor_SMD:R_0603_1608Metric -> Resistor_SMD:R_0603_1608Metric_Pad1.05x0.95mm_HandSolder
- R3: renamed from R6; footprint Resistor_SMD:R_0603_1608Metric -> Resistor_SMD:R_0603_1608Metric_Pad1.05x0.95mm_HandSolder
- R5: renamed from R7; footprint Resistor_SMD:R_0603_1608Metric -> Resistor_SMD:R_0603_1608Metric_Pad1.05x0.95mm_HandSolder
- R7: renamed from R9; footprint Resistor_SMD:R_0603_1608Metric -> Resistor_SMD:R_0603_1608Metric_Pad1.05x0.95mm_HandSolder
- R9: renamed from R2; footprint Resistor_SMD:R_0603_1608Metric -> Resistor_SMD:R_0603_1608Metric_Pad1.05x0.95mm_HandSolder
Connections:
- net +5V: now also J7'1.5 (Pin_5), SW1.2, SW2.2
- net 1Wire-1: now also XA1.D47; no longer XA1.D31
- net 1Wire-2: now also XA1.D29; no longer XA1.D37
- net 1Wire-3: now also XA1.D28; no longer XA1.D35
- net DHT22-1: now also XA1.D45; no longer XA1.D27
- net DHT22-2: now also XA1.D35; no longer XA1.D41
- net DHT22-3: now also XA1.D36; no longer XA1.D33
- net GND: now also C1.2, C2.2, C3.2, C4.2, J7'1.4 (Pin_4), R12.2, R13.2, R14.2, R15.2, R16.2, R17.2, R18.2, R19.2
- net INA1: now also C1.1, R2.2; no longer U1.1
- net INA2: now also XA1.A3, C2.1, R4.2; no longer U2.1, XA1.A2
- net INA3: now also XA1.A5, C3.1, R6.2; no longer U3.1, XA1.A3
- net INA4: now also XA1.A7, C4.1, R8.2; no longer U4.1, XA1.A4
- net RX3: now also J7'1.3 (Pin_3)
- net SPI-SS-Pressure-1: now also XA1.D33; no longer XA1.D39
- net SPI-SS-Pressure-2: now also XA1.D48; no longer XA1.D25
- net TX3: now also J7'1.2 (Pin_2)
- net DC-Pump-2: now reaches XA1.A6
- net DC-Pump-2: now also J3.4 (Pin_4)
- net LED-1: now reaches XA1.D2 (D2_INT0)
- net LED-1: now also D1.2 (A)
- net LED-2: now reaches XA1.D3 (D3_INT1)
- net LED-2: now also D2.2 (A)
- net Button-1: now reaches XA1.D32
- net Button-1: now also R12.1, SW1.1
- net LED-3: now reaches XA1.D4
- net LED-3: now also D3.2 (A)
- net Button-2: now reaches XA1.D40
- net Button-2: now also R13.1, SW2.1
- net LED-4: now reaches XA1.D5
- net LED-4: now also D4.2 (A)
- net LED-5: now reaches XA1.D6
- net LED-5: now also D5.2 (A)
- net LED-6: now reaches XA1.D7
- net LED-6: now also D6.2 (A)
- net DC-Servo: now reaches J5.4 (Pin_4)
- net DC-Servo: now also XA1.A2
- net DC-Pump-1: now reaches J2.4 (Pin_4)
- net DC-Pump-1: now also XA1.A4
- net Pump-GPIO: no longer names the net of DSUB-Servo1.3
- net Pump-GPIO: no longer XA1.D29
- new net: R2.1, U1.1
- new net: R6.1, U3.1
- new net: R8.1, U4.1
- new net: R4.1, U2.1
- new net: D1.1 (K), R14.1
- new net: D2.1 (K), R15.1
- new net: D3.1 (K), R16.1
- new net: D4.1 (K), R17.1
- new net: D5.1 (K), R18.1
- new net: D6.1 (K), R19.1
Other:
- note added: "R = T/(Tau * C) \n"
- moved on the sheet: J1, J2, J3, J4, J5, R1, R3, R5, R7, U1, U2, U3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
