File: mech/mech.sch (KiCad schematic (older format))
At the start: 24 parts, among them P1 Pump_Motor_DC, P2 Pump_Motor_DC, T1 DS18B20, T2 DS18B20, U1 DHT22

Commit message: ADC + PCA9685 version
Parts:
- removed D2: LED, LED_SMD:LED_0402_1005Metric, symbol Device:LED
- removed DSUB1: DB25_Female, Connector_Dsub:DSUB-25_Female_Horizontal_P2.77x2.54mm_EdgePinOffset9.40mm, symbol Connector:DB25_Female
- removed R820: R, Resistor_SMD:R_0402_1005Metric, symbol Device:R
- added ADC1, ADC2: MAX11615, Package_SO:QSOP-16_3.9x4.9mm_P0.635mm, symbol Analog_ADC:MAX11615
- added DSUB1: DB9_Female, symbol Connector:DB9_Female_MountingHoles
- added R10k1: R, symbol Device:R
- added RV1, RV10, RV11, RV12, RV13, RV14, RV2, RV3, RV4, RV5, RV6, RV7, RV8, RV9: R_POT, Connector_PinHeader_2.54mm:PinHeader_1x03_P2.54mm_Vertical, symbol Device:R_POT
- added U2: PCA9685PW, Package_SO:TSSOP-28_4.4x9.7mm_P0.65mm, symbol Driver_LED:PCA9685PW
Connections:
- net labels added: 1Wire, DHT22, I2C-SCL, I2C-SDA, Pump-1, Pump-2
- net labels removed: +12V
- wire segments 121 -> 156
Other:
- moved on the sheet: D1, M-1, M-10, M-11, M-12, M-13, M-14, M-2, M-3, M-4, M-5, M-6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

Commit message: mumble
Parts:
- removed ADC1, ADC2: MAX11615, Package_SO:QSOP-16_3.9x4.9mm_P0.635mm, symbol Analog_ADC:MAX11615
- removed D1: LED, LED_SMD:LED_0402_1005Metric, symbol Device:LED
- removed R330: R, Resistor_SMD:R_0402_1005Metric, symbol Device:R
- added C0, C6: C100nF, Resistor_SMD:R_0603_1608Metric, symbol Device:C
- added C2: 10nF, Resistor_SMD:R_0603_1608Metric, symbol Device:C
- added C3: 100nF, Resistor_SMD:R_0603_1608Metric, symbol Device:C
- added C5: C10nF, Resistor_SMD:R_0603_1608Metric, symbol Device:C
- added R10k2: R, Resistor_SMD:R_0603_1608Metric, symbol Device:R
- added U3, U4: ADC128D818, Package_SO:TSSOP-16_4.4x5mm_P0.65mm, symbol Analog_ADC:ADC128D818
- DSUB1: footprint (none) -> Connector_Dsub:DSUB-9_Female_Horizontal_P2.77x2.84mm_EdgePinOffset4.94mm_Housed_MountingHolesOffset7.48mm
- R10k1: footprint (none) -> Resistor_SMD:R_0603_1608Metric
Connections:
- net labels added: addr:0011101b:1Dh, addr:0110111b:37h
- wire segments 156 -> 197
Other:
- moved on the sheet: P1, P2, RV1, RV10, RV11, RV2, RV3, RV4, RV9

Commit message: final
Parts:
- added C1, C4: C100nF, Resistor_SMD:R_0603_1608Metric, symbol Device:C
- renumbered RV5 to RV1, RV9 to RV10, RV1 to RV11, RV4 to RV12, RV3 to RV13, RV2 to RV14, RV6 to RV2, RV7 to RV3, RV8 to RV4, RV12 to RV5, RV13 to RV6, RV14 to RV7, RV11 to RV8, RV10 to RV9
Connections:
- wire segments 197 -> 203
Other:
- moved on the sheet: P1, P2, T1, T2, U1

Commit message: move mosfet to mech board, controll pump via gnd
Parts:
- added U5, U6: IRFL210, Package_TO_SOT_SMD:SOT-223, symbol irfl210:IRFL210
Connections:
- net labels added: +12V, Pump, Pump-1-2
- net labels removed: Pump-1, Pump-2
- wire segments 203 -> 207
Other:
- moved on the sheet: P1
Changed lines of the file:
@@
 L Motor:Motor_DC P1
 U 1 1 5EE707F5
-P 2800 5600
-F 0 "P1" H 2958 5596 50  0000 L CNN
-F 1 "Pump_Motor_DC" H 2958 5505 50  0000 L CNN
-F 2 "Connector_JST:JST_EH_B2B-EH-A_1x02_P2.50mm_Vertical" H 2800 5510 50  0001 C CNN
-F 3 "~" H 2800 5510 50  0001 C CNN
-	1    2800 5600
+P 3200 5600
+F 0 "P1" H 3358 5596 50  0000 L CNN
+F 1 "Pump_Motor_DC" H 3358 5505 50  0000 L CNN
+F 2 "Connector_JST:JST_EH_B2B-EH-A_1x02_P2.50mm_Vertical" H 3200 5510 50  0001 C CNN
+F 3 "~" H 3200 5510 50  0001 C CNN
+	1    3200 5600
 	1    0    0    -1
 $EndComp
@@
 L power:GND #PWR0150
 U 1 1 5EE90E71
-P 2800 5900
-F 0 "#PWR0150" H 2800 5650 50  0001 C CNN
-F 1 "GND" H 2805 5727 50  0000 C CNN
-F 2 "" H 2800 5900 50  0001 C CNN
-F 3 "" H 2800 5900 50  0001 C CNN
-	1    2800 5900
-	1    0    0    -1
-$EndComp
-$Comp
-L power:GND #PWR0153
-U 1 1 5EEB29F5
-P 1700 5900
-F 0 "#PWR0153" H 1700 5650 50  0001 C CNN
-F 1 "GND" H 1705 5727 50  0000 C CNN
-F 2 "" H 1700 5900 50  0001 C CNN
-F 3 "" H 1700 5900 50  0001 C CNN
-	1    1700 5900
+P 3200 6500
+F 0 "#PWR0150" H 3200 6250 50  0001 C CNN
+F 1 "GND" H 3205 6327 50  0000 C CNN
+F 2 "" H 3200 6500 50  0001 C CNN
+F 3 "" H 3200 6500 50  0001 C CNN
+	1    3200 6500
 	1    0    0    -1
 $EndComp
@@
 	1    0    0    -1
 $EndComp
-Text GLabel 1700 5300 1    50   Input ~ 0
-Pump-1
-Text GLabel 2800 5300 1    50   Input ~ 0
-Pump-2
 Wire Wire Line
 	7750 8850 7750 9000
@@
 	2100 9350 2100 11050
 Wire Wire Line
-	2800 5300 2800 5400
+	3200 5300 3200 5400
 $Comp
 L power:+5V #PWR0187
@@
 	1    0    0    -1
 $EndComp
-Text GLabel 3150 2250 2    50   Input ~ 0
-Pump-1
 Wire Wire Line
 	3350 2150 3350 1950
@@
 Wire Wire Line
 	3150 2950 3350 2950
-Text GLabel 3150 2850 2    50   Input ~ 0
-Pump-2
 Wire Wire Line
 	4500 5100 4500 5200
@@
 Wire Wire Line
 	2850 8400 2850 9150
+Wire Wire Line
+	3750 2250 3750 2050
+Wire Wire Line
+	3150 2250 3750 2250
+$Comp
+L power:+12V #PWR0153
+U 1 1 5EA8ED54
+P 3750 2050
+F 0 "#PWR0153" H 3750 1900 50  0001 C CNN
+F 1 "+12V" H 3765 2223 50  0000 C CNN
+F 2 "" H 3750 2050 50  0001 C CNN
+F 3 "" H 3750 2050 50  0001 C CNN
+	1    3750 2050
+	1    0    0    -1
+$EndComp
+Wire Wire Line
+	3750 2850 3750 2650
+Wire Wire Line
+	3150 2850 3750 2850
+$Comp
+L power:+12V #PWR0183
+U 1 1 5EAD8EE8
+P 3750 2650
+F 0 "#PWR0183" H 3750 2500 50  0001 C CNN
+F 1 "+12V" H 3765 2823 50  0000 C CNN
+F 2 "" H 3750 2650 50  0001 C CNN
+F 3 "" H 3750 2650 50  0001 C CNN
+	1    3750 2650
+	1    0    0    -1
+$EndComp
+Text GLabel 2900 6200 0    50   Input ~ 0
+Pump
+$Comp
+L power:+12V #PWR0190
+U 1 1 5EB4C830
+P 1700 5300
+F 0 "#PWR0190" H 1700 5150 50  0001 C CNN
+F 1 "+12V" H 1715 5473 50  0000 C CNN
+F 2 "" H 1700 5300 50  0001 C CNN
+F 3 "" H 1700 5300 50  0001 C CNN
+	1    1700 5300
+	1    0    0    -1
+$EndComp
+$Comp
+L power:+12V #PWR0191
+U 1 1 5EB5A510
+P 3200 5300
+F 0 "#PWR0191" H 3200 5150 50  0001 C CNN
+F 1 "+12V" H 3215 5473 50  0000 C CNN
+F 2 "" H 3200 5300 50  0001 C CNN
+F 3 "" H 3200 5300 50  0001 C CNN
+	1    3200 5300
+	1    0    0    -1
+$EndComp
+$Comp
+L power:GND #PWR0192
+U 1 1 5EB985C1
+P 1700 6500
+F 0 "#PWR0192" H 1700 6250 50  0001 C CNN
+F 1 "GND" H 1705 6327 50  0000 C CNN
+F 2 "" H 1700 6500 50  0001 C CNN
+F 3 "" H 1700 6500 50  0001 C CNN
+	1    1700 6500
+	1    0    0    -1
+$EndComp
+$Comp
+L irfl210:IRFL210 U5
+U 1 1 5EB985C7
+P 2000 6200
+F 0 "U5" V 2046 6422 50  0000 R CNN
+F 1 "IRFL210" V 1955 6422 50  0000 R CNN
+F 2 "Package_TO_SOT_SMD:SOT-223" H 2000 6350 50  0001 C CNN
+F 3 "https://sensing.honeywell.com/index.php?ci_id=151134" H 2000 6150 50  0001 C CNN
+	1    2000 6200
+	0    -1   -1   0
+$EndComp
+$Comp
+L irfl210:IRFL210 U6
+U 1 1 5EB68DC6
+P 3500 6200
+F 0 "U6" V 3546 6422 50  0000 R CNN
+F 1 "IRFL210" V 3455 6422 50  0000 R CNN
+F 2 "Package_TO_SOT_SMD:SOT-223" H 3500 6350 50  0001 C CNN
+F 3 "https://sensing.honeywell.com/index.php?ci_id=151134" H 3500 6150 50  0001 C CNN
+	1    3500 6200
+	0    -1   -1   0
+$EndComp
+Text GLabel 3150 2550 2    50   Input ~ 0
+Pump-1-2
+Text GLabel 1400 6200 0    50   Input ~ 0
+Pump
 $EndSCHEMATC

Commit message: add db9 models, and update footprints
Parts:
- DSUB1: value DB9_Female -> DB9_Male; footprint Connector_Dsub:DSUB-9_Female_Horizontal_P2.77x2.84mm_EdgePinOffset4.94mm_Housed_MountingHolesOffset7.48mm -> Connector_Dsub:DSUB-9_Male_Horizontal_P2.77x2.84mm_EdgePinOffset7.70mm_Housed_MountingHolesOffset9.12mm; symbol Connector:DB9_Female_MountingHoles -> Connector:DB9_Male_MountingHoles
Changed lines of the file:
@@
 encoding utf-8
 Sheet 1 1
-Title ""
-Date ""
-Rev ""
-Comp ""
+Title "Stardust Mech PCB"
+Date "27 April 2020"
+Rev "1.0"
+Comp "Stardust"
 Comment1 ""
 Comment2 ""
@@
 	7850 9750 6750 9750
 $Comp
-L Connector:DB9_Female_MountingHoles DSUB1
+L Connector:DB9_Male_MountingHoles DSUB1
 U 1 1 5F245498
 P 2850 2550
 F 0 "DSUB1" H 3030 2459 50  0000 L CNN
-F 1 "DB9_Female" H 3030 2550 50  0000 L CNN
-F 2 "Connector_Dsub:DSUB-9_Female_Horizontal_P2.77x2.84mm_EdgePinOffset4.94mm_Housed_MountingHolesOffset7.48mm" H 2850 2550 50  0001 C CNN
+F 1 "DB9_Male" H 3030 2550 50  0000 L CNN
+F 2 "Connector_Dsub:DSUB-9_Male_Horizontal_P2.77x2.84mm_EdgePinOffset7.70mm_Housed_MountingHolesOffset9.12mm" H 2850 2550 50  0001 C CNN
 F 3 " ~" H 2850 2550 50  0001 C CNN
 	1    2850 2550

Commit message: rev.2 init
Parts:
- added D1, D2: LED, Resistor_SMD:R_0603_1608Metric_Pad1.05x0.95mm_HandSolder, symbol Device:LED
- added R1, R2: 1k, Resistor_SMD:R_0603_1608Metric_Pad1.05x0.95mm_HandSolder, symbol Device:R
- C0, C1, C2, C3, C4, C5, C6, R10k1, R10k2: footprint Resistor_SMD:R_0603_1608Metric -> Resistor_SMD:R_0603_1608Metric_Pad1.05x0.95mm_HandSolder
Connections:
- net +12V: now also D1.1 (K), D2.1 (K)
- net at P1.2 (-), U6.2 (D): now also R1.2
- net at P2.2 (-), U5.2 (D): now also R2.2
- new net: D2.2 (A), R2.1
- new net: D1.2 (A), R1.1
Other:
- moved on the sheet: P2
Changed lines of the file:
@@
 $EndDescr
-$Comp
-L Motor:Motor_DC P1
-U 1 1 5EE707F5
-P 3200 5600
-F 0 "P1" H 3358 5596 50  0000 L CNN
-F 1 "Pump_Motor_DC" H 3358 5505 50  0000 L CNN
-F 2 "Connector_JST:JST_EH_B2B-EH-A_1x02_P2.50mm_Vertical" H 3200 5510 50  0001 C CNN
-F 3 "~" H 3200 5510 50  0001 C CNN
-	1    3200 5600
-	1    0    0    -1
-$EndComp
-$Comp
-L power:GND #PWR0150
-U 1 1 5EE90E71
-P 3200 6500
-F 0 "#PWR0150" H 3200 6250 50  0001 C CNN
-F 1 "GND" H 3205 6327 50  0000 C CNN
-F 2 "" H 3200 6500 50  0001 C CNN
-F 3 "" H 3200 6500 50  0001 C CNN
-	1    3200 6500
-	1    0    0    -1
-$EndComp
 $Comp
 L Motor:Motor_DC P2
 U 1 1 5EEB29E8
-P 1700 5600
-F 0 "P2" H 1858 5596 50  0000 L CNN
-F 1 "Pump_Motor_DC" H 1858 5505 50  0000 L CNN
-F 2 "Connector_JST:JST_EH_B2B-EH-A_1x02_P2.50mm_Vertical" H 1700 5510 50  0001 C CNN
-F 3 "~" H 1700 5510 50  0001 C CNN
-	1    1700 5600
+P 1900 5500
+F 0 "P2" H 2058 5496 50  0000 L CNN
+F 1 "Pump_Motor_DC" H 2058 5405 50  0000 L CNN
+F 2 "Connector_JST:JST_EH_B2B-EH-A_1x02_P2.50mm_Vertical" H 1900 5410 50  0001 C CNN
+F 3 "~" H 1900 5410 50  0001 C CNN
+	1    1900 5500
 	1    0    0    -1
 $EndComp
@@
 $EndComp
 Wire Wire Line
-	1700 5300 1700 5400
+	1700 5150 1700 5250
 Text GLabel 3150 2750 2    50   Input ~ 0
 1Wire
@@
 F 0 "C0" H 5715 4246 50  0000 L CNN
 F 1 "C100nF" H 5715 4155 50  0000 L CNN
-F 2 "Resistor_SMD:R_0603_1608Metric" H 5638 4050 50  0001 C CNN
+F 2 "Resistor_SMD:R_0603_1608Metric_Pad1.05x0.95mm_HandSolder" H 5638 4050 50  0001 C CNN
 F 3 "~" H 5600 4200 50  0001 C CNN
 	1    5600 4200
@@
 F 0 "R10k1" H 1800 8500 50  0000 L CNN
 F 1 "R" H 1900 8400 50  0000 L CNN
-F 2 "Resistor_SMD:R_0603_1608Metric" V 2030 8450 50  0001 C CNN
+F 2 "Resistor_SMD:R_0603_1608Metric_Pad1.05x0.95mm_HandSolder" V 2030 8450 50  0001 C CNN
 F 3 "~" H 2100 8450 50  0001 C CNN
 	1    2100 8450
@@
 F 0 "R10k2" H 2270 8796 50  0000 L CNN
 F 1 "R" H 2350 8700 50  0000 L CNN
-F 2 "Resistor_SMD:R_0603_1608Metric" V 2130 8750 50  0001 C CNN
+F 2 "Resistor_SMD:R_0603_1608Metric_Pad1.05x0.95mm_HandSolder" V 2130 8750 50  0001 C CNN
 F 3 "~" H 2200 8750 50  0001 C CNN
 	1    2200 8750
@@
 F 0 "C5" H 3750 14600 50  0000 L CNN
 F 1 "C10nF" H 3750 14450 50  0000 L CNN
-F 2 "Resistor_SMD:R_0603_1608Metric" H 4088 14400 50  0001 C CNN
+F 2 "Resistor_SMD:R_0603_1608Metric_Pad1.05x0.95mm_HandSolder" H 4088 14400 50  0001 C CNN
 F 3 "~" H 4050 14550 50  0001 C CNN
 	1    4050 14550
@@
 Wire Wire Line
 	2100 9350 2100 11050
-Wire Wire Line
-	3200 5300 3200 5400
 $Comp
 L power:+5V #PWR0187
@@
 F 0 "C3" H 4415 10646 50  0000 L CNN
 F 1 "100nF" H 4400 10500 50  0000 L CNN
-F 2 "Resistor_SMD:R_0603_1608Metric" H 4338 10450 50  0001 C CNN
+F 2 "Resistor_SMD:R_0603_1608Metric_Pad1.05x0.95mm_HandSolder" H 4338 10450 50  0001 C CNN
 F 3 "~" H 4300 10600 50  0001 C CNN
 	1    4300 10600
@@
 F 0 "C2" H 3750 10650 50  0000 L CNN
 F 1 "10nF" H 3750 10500 50  0000 L CNN
-F 2 "Resistor_SMD:R_0603_1608Metric" H 4088 10450 50  0001 C CNN
+F 2 "Resistor_SMD:R_0603_1608Metric_Pad1.05x0.95mm_HandSolder" H 4088 10450 50  0001 C CNN
 F 3 "~" H 4050 10600 50  0001 C CNN
 	1    4050 10600
@@
 F 0 "C6" H 4415 14596 50  0000 L CNN
 F 1 "C100nF" H 4400 14450 50  0000 L CNN
-F 2 "Resistor_SMD:R_0603_1608Metric" H 4338 14400 50  0001 C CNN
+F 2 "Resistor_SMD:R_0603_1608Metric_Pad1.05x0.95mm_HandSolder" H 4338 14400 50  0001 C CNN
 F 3 "~" H 4300 14550 50  0001 C CNN
 	1    4300 14550
@@
 F 0 "C4" H 3165 12646 50  0000 L CNN
 F 1 "C100nF" H 3150 12500 50  0000 L CNN
-F 2 "Resistor_SMD:R_0603_1608Metric" H 3088 12450 50  0001 C CNN
+F 2 "Resistor_SMD:R_0603_1608Metric_Pad1.05x0.95mm_HandSolder" H 3088 12450 50  0001 C CNN
 F 3 "~" H 3050 12600 50  0001 C CNN
 	1    3050 12600
@@
 F 0 "C1" H 3165 8696 50  0000 L CNN
 F 1 "C100nF" H 3150 8550 50  0000 L CNN
-F 2 "Resistor_SMD:R_0603_1608Metric" H 3088 8500 50  0001 C CNN
+F 2 "Resistor_SMD:R_0603_1608Metric_Pad1.05x0.95mm_HandSolder" H 3088 8500 50  0001 C CNN
 F 3 "~" H 3050 8650 50  0001 C CNN
 	1    3050 8650
@@
 	1    0    0    -1
 $EndComp
-Text GLabel 2900 6200 0    50   Input ~ 0
-Pump
 $Comp
 L power:+12V #PWR0190
 U 1 1 5EB4C830
-P 1700 5300
-F 0 "#PWR0190" H 1700 5150 50  0001 C CNN
-F 1 "+12V" H 1715 5473 50  0000 C CNN
-F 2 "" H 1700 5300 50  0001 C CNN
-F 3 "" H 1700 5300 50  0001 C CNN
-	1    1700 5300
-	1    0    0    -1
-$EndComp
-$Comp
-L power:+12V #PWR0191
-U 1 1 5EB5A510
-P 3200 5300
-F 0 "#PWR0191" H 3200 5150 50  0001 C CNN
-F 1 "+12V" H 3215 5473 50  0000 C CNN
-F 2 "" H 3200 5300 50  0001 C CNN
-F 3 "" H 3200 5300 50  0001 C CNN
-	1    3200 5300
+P 1700 5150
+F 0 "#PWR0190" H 1700 5000 50  0001 C CNN
+F 1 "+12V" H 1715 5323 50  0000 C CNN
+F 2 "" H 1700 5150 50  0001 C CNN
+F 3 "" H 1700 5150 50  0001 C CNN
+	1    1700 5150
 	1    0    0    -1
 $EndComp
@@
 	0    -1   -1   0
 $EndComp
-$Comp
-L irfl210:IRFL210 U6
-U 1 1 5EB68DC6
-P 3500 6200
-F 0 "U6" V 3546 6422 50  0000 R CNN
-F 1 "IRFL210" V 3455 6422 50  0000 R CNN
-F 2 "Package_TO_SOT_SMD:SOT-223" H 3500 6350 50  0001 C CNN
-F 3 "https://sensing.honeywell.com/index.php?ci_id=151134" H 3500 6150 50  0001 C CNN
-	1    3500 6200
-	0    -1   -1   0
-$EndComp
 Text GLabel 3150 2550 2    50   Input ~ 0
 Pump-1-2
 Text GLabel 1400 6200 0    50   Input ~ 0
 Pump
+$Comp
+L Device:LED D2
+U 1 1 5EAEB45E
+P 1500 5400
+F 0 "D2" V 1447 5478 50  0000 L CNN
+F 1 "LED" V 1538 5478 50  0000 L CNN
+F 2 "Resistor_SMD:R_0603_1608Metric_Pad1.05x0.95mm_HandSolder" H 1500 5400 50  0001 C CNN
+F 3 "~" H 1500 5400 50  0001 C CNN
+	1    1500 5400
+	0    1    1    0
+$EndComp
+Wire Wire Line
+	1700 5900 1700 5850
+Wire Wire Line
+	1700 5850 1900 5850
+Wire Wire Line
+	1900 5850 1900 5800
+Wire Wire Line
+	1700 5850 1500 5850
+Connection ~ 1700 5850
+Wire Wire Line
+	1500 5250 1700 5250
+Wire Wire Line
+	1900 5300 1900 5250
+Wire Wire Line
+	1900 5250 1700 5250
+Connection ~ 1700 5250
+$Comp
+L Device:R R2
+U 1 1 5EBD701E
+P 1500 5700
+F 0 "R2" H 1570 5746 50  0000 L CNN
+F 1 "1k" H 1570 5655 50  0000 L CNN
+F 2 "Resistor_SMD:R_0603_1608Metric_Pad1.05x0.95mm_HandSolder" V 1430 5700 50  0001 C CNN
+F 3 "~" H 1500 5700 50  0001 C CNN
+	1    1500 5700
+	1    0    0    -1
+$EndComp
+$Comp
+L Motor:Motor_DC P1
+U 1 1 5EC06134
+P 3350 5500
+F 0 "P1" H 3508 5496 50  0000 L CNN
+F 1 "Pump_Motor_DC" H 3508 5405 50  0000 L CNN
+F 2 "Connector_JST:JST_EH_B2B-EH-A_1x02_P2.50mm_Vertical" H 3350 5410 50  0001 C CNN
+F 3 "~" H 3350 5410 50  0001 C CNN
+	1    3350 5500
+	1    0    0    -1
+$EndComp
+Wire Wire Line
+	3150 5150 3150 5250
+$Comp
+L power:+12V #PWR0150
+U 1 1 5EC0613B
+P 3150 5150
+F 0 "#PWR0150" H 3150 5000 50  0001 C CNN
+F 1 "+12V" H 3165 5323 50  0000 C CNN
+F 2 "" H 3150 5150 50  0001 C CNN
+F 3 "" H 3150 5150 50  0001 C CNN
+	1    3150 5150
+	1    0    0    -1
+$EndComp
+$Comp
+L power:GND #PWR0191
+U 1 1 5EC06141
+P 3150 6500
+F 0 "#PWR0191" H 3150 6250 50  0001 C CNN
+F 1 "GND" H 3155 6327 50  0000 C CNN
+F 2 "" H 3150 6500 50  0001 C CNN
+F 3 "" H 3150 6500 50  0001 C CNN
+	1    3150 6500
+	1    0    0    -1
+$EndComp
+$Comp
+L irfl210:IRFL210 U6
+U 1 1 5EC06147
+P 3450 6200
+F 0 "U6" V 3496 6422 50  0000 R CNN
+F 1 "IRFL210" V 3405 6422 50  0000 R CNN
+F 2 "Package_TO_SOT_SMD:SOT-223" H 3450 6350 50  0001 C CNN
+F 3 "https://sensing.honeywell.com/index.php?ci_id=151134" H 3450 6150 50  0001 C CNN
+	1    3450 6200
+	0    -1   -1   0
+$EndComp
+Text GLabel 2850 6200 0    50   Input ~ 0
+Pump
+$Comp
+L Device:LED D1
+U 1 1 5EC0614E
+P 2950 5400
+F 0 "D1" V 2897 5478 50  0000 L CNN
+F 1 "LED" V 2988 5478 50  0000 L CNN
+F 2 "Resistor_SMD:R_0603_1608Metric_Pad1.05x0.95mm_HandSolder" H 2950 5400 50  0001 C CNN
+F 3 "~" H 2950 5400 50  0001 C CNN
+	1    2950 5400
+	0    1    1    0
+$EndComp
+Wire Wire Line
+	3150 5900 3150 5850
+Wire Wire Line
+	3150 5850 3350 5850
+Wire Wire Line
+	3350 5850 3350 5800
+Wire Wire Line
+	3150 5850 2950 5850
+Connection ~ 3150 5850
+Wire Wire Line
+	2950 5250 3150 5250
+Wire Wire Line
+	3350 5300 3350 5250
+Wire Wire Line
+	3350 5250 3150 5250
+Connection ~ 3150 5250
+$Comp
+L Device:R R1
+U 1 1 5EC0615D
+P 2950 5700
+F 0 "R1" H 3020 5746 50  0000 L CNN
+F 1 "1k" H 3020 5655 50  0000 L CNN
+F 2 "Resistor_SMD:R_0603_1608Metric_Pad1.05x0.95mm_HandSolder" V 2880 5700 50  0001 C CNN
+F 3 "~" H 2950 5700 50  0001 C CNN
+	1    2950 5700
+	1    0    0    -1
+$EndComp
 $EndSCHEMATC

Commit message: mech pcb tweaks
Parts:
- removed U5, U6: IRFL210, Package_TO_SOT_SMD:SOT-223, symbol irfl210:IRFL210
Connections:
- net Pump-1-2 is gone; now on net GND: DSUB1.3
- net GND: now also P1.2 (-), P2.2 (-), R1.2, R2.2
Changed lines of the file:
@@
 	3150 2150 3350 2150
 Wire Wire Line
-	3350 3150 3350 2950
+	3600 3150 3600 2950
 $Comp
 L power:GND #PWR0116
 U 1 1 5F75D03D
-P 3350 3150
-F 0 "#PWR0116" H 3350 2900 50  0001 C CNN
-F 1 "GND" H 3355 2977 50  0000 C CNN
-F 2 "" H 3350 3150 50  0001 C CNN
-F 3 "" H 3350 3150 50  0001 C CNN
-	1    3350 3150
-	1    0    0    -1
-$EndComp
-Wire Wire Line
-	3150 2950 3350 2950
+P 3600 3150
+F 0 "#PWR0116" H 3600 2900 50  0001 C CNN
+F 1 "GND" H 3605 2977 50  0000 C CNN
+F 2 "" H 3600 3150 50  0001 C CNN
+F 3 "" H 3600 3150 50  0001 C CNN
+	1    3600 3150
+	1    0    0    -1
+$EndComp
 Wire Wire Line
 	4500 5100 4500 5200
@@
 $EndComp
 Wire Wire Line
-	3750 2850 3750 2650
-Wire Wire Line
 	3150 2850 3750 2850
-$Comp
-L power:+12V #PWR0183
-U 1 1 5EAD8EE8
-P 3750 2650
-F 0 "#PWR0183" H 3750 2500 50  0001 C CNN
-F 1 "+12V" H 3765 2823 50  0000 C CNN
-F 2 "" H 3750 2650 50  0001 C CNN
-F 3 "" H 3750 2650 50  0001 C CNN
-	1    3750 2650
-	1    0    0    -1
-$EndComp
 $Comp
 L power:+12V #PWR0190
@@
 L power:GND #PWR0192
 U 1 1 5EB985C1
-P 1700 6500
-F 0 "#PWR0192" H 1700 6250 50  0001 C CNN
-F 1 "GND" H 1705 6327 50  0000 C CNN
-F 2 "" H 1700 6500 50  0001 C CNN
-F 3 "" H 1700 6500 50  0001 C CNN
-	1    1700 6500
-	1    0    0    -1
-$EndComp
-$Comp
-L irfl210:IRFL210 U5
-U 1 1 5EB985C7
-P 2000 6200
-F 0 "U5" V 2046 6422 50  0000 R CNN
-F 1 "IRFL210" V 1955 6422 50  0000 R CNN
-F 2 "Package_TO_SOT_SMD:SOT-223" H 2000 6350 50  0001 C CNN
-F 3 "https://sensing.honeywell.com/index.php?ci_id=151134" H 2000 6150 50  0001 C CNN
-	1    2000 6200
-	0    -1   -1   0
-$EndComp
-Text GLabel 3150 2550 2    50   Input ~ 0
-Pump-1-2
-Text GLabel 1400 6200 0    50   Input ~ 0
-Pump
+P 1700 6050
+F 0 "#PWR0192" H 1700 5800 50  0001 C CNN
+F 1 "GND" H 1705 5877 50  0000 C CNN
+F 2 "" H 1700 6050 50  0001 C CNN
+F 3 "" H 1700 6050 50  0001 C CNN
+	1    1700 6050
+	1    0    0    -1
+$EndComp
 $Comp
 L Device:LED D2
@@
 $EndComp
 Wire Wire Line
-	1700 5900 1700 5850
-Wire Wire Line
 	1700 5850 1900 5850
 Wire Wire Line
@@
 L power:GND #PWR0191
 U 1 1 5EC06141
-P 3150 6500
-F 0 "#PWR0191" H 3150 6250 50  0001 C CNN
-F 1 "GND" H 3155 6327 50  0000 C CNN
-F 2 "" H 3150 6500 50  0001 C CNN
-F 3 "" H 3150 6500 50  0001 C CNN
-	1    3150 6500
-	1    0    0    -1
-$EndComp
-$Comp
-L irfl210:IRFL210 U6
-U 1 1 5EC06147
-P 3450 6200
-F 0 "U6" V 3496 6422 50  0000 R CNN
-F 1 "IRFL210" V 3405 6422 50  0000 R CNN
-F 2 "Package_TO_SOT_SMD:SOT-223" H 3450 6350 50  0001 C CNN
-F 3 "https://sensing.honeywell.com/index.php?ci_id=151134" H 3450 6150 50  0001 C CNN
-	1    3450 6200
-	0    -1   -1   0
-$EndComp
-Text GLabel 2850 6200 0    50   Input ~ 0
-Pump
+P 3150 6050
+F 0 "#PWR0191" H 3150 5800 50  0001 C CNN
+F 1 "GND" H 3155 5877 50  0000 C CNN
+F 2 "" H 3150 6050 50  0001 C CNN
+F 3 "" H 3150 6050 50  0001 C CNN
+	1    3150 6050
+	1    0    0    -1
+$EndComp
 $Comp
 L Device:LED D1
@@
 $EndComp
 Wire Wire Line
-	3150 5900 3150 5850
-Wire Wire Line
 	3150 5850 3350 5850
 Wire Wire Line
@@
 	1    0    0    -1
 $EndComp
+Wire Wire Line
+	3150 5850 3150 6050
+Wire Wire Line
+	1700 5850 1700 6050
+Wire Wire Line
+	3150 2950 3600 2950
+Wire Wire Line
+	3600 2950 3600 2550
+Wire Wire Line
+	3600 2550 3150 2550
+Connection ~ 3600 2950
+Wire Wire Line
+	3750 2250 3750 2850
+Connection ~ 3750 2250
 $EndSCHEMATC
