File: sensor/sensor.sch (KiCad schematic (older format))
At the start: 5 parts, among them T1 DS18B20, T2 DS18B20, U1 DHT22, U9 SSCDRNN015PASA5

Commit message: modifications
Parts:
- renumbered DSUB1 to DSUB2
Connections:
- net labels added: SPI-MISO, SPI-MOSI
- net labels removed: SPI-SDA, SPI-SDO
- wire segments 9 -> 7
Changed lines of the file:
@@
 DHT22
 $Comp
-L Connector:DB9_Female_MountingHoles DSUB1
+L Connector:DB9_Female_MountingHoles DSUB2
 U 1 1 5F245498
 P 3600 3400
-F 0 "DSUB1" H 3780 3309 50  0000 L CNN
+F 0 "DSUB2" H 3780 3309 50  0000 L CNN
 F 1 "DB9_Female" H 3780 3400 50  0000 L CNN
 F 2 "Connector_Dsub:DSUB-9_Female_Horizontal_P2.77x2.84mm_EdgePinOffset4.94mm_Housed_MountingHolesOffset7.48mm" H 3600 3400 50  0001 C CNN
@@
 	1    0    0    -1
 $EndComp
-Text GLabel 7500 4100 2    50   Input ~ 0
-SPI-SDA
-Wire Wire Line
-	8050 3900 8050 4000
-$Comp
-L power:GND #PWR0154
-U 1 1 5EEF4069
-P 8050 4000
-F 0 "#PWR0154" H 8050 3750 50  0001 C CNN
-F 1 "GND" H 8055 3827 50  0000 C CNN
-F 2 "" H 8050 4000 50  0001 C CNN
-F 3 "" H 8050 4000 50  0001 C CNN
-	1    8050 4000
-	1    0    0    -1
-$EndComp
 Text GLabel 7500 4300 2    50   Input ~ 0
 SPI-SS-Pressure
@@
 	1    0    0    -1
 $EndComp
-Wire Wire Line
-	7500 3900 8050 3900
 Text GLabel 3900 3400 2    50   Input ~ 0
-SPI-SDO
+SPI-MISO
 Text GLabel 3900 3500 2    50   Input ~ 0
 SPI-SS-Pressure
@@
 	-1   0    0    -1
 $EndComp
-Text GLabel 3900 3700 2    50   Input ~ 0
-SPI-SDA
 Text GLabel 3900 3300 2    50   Input ~ 0
 SPI-CLK
 Text GLabel 7500 4000 2    50   Input ~ 0
+SPI-MISO
+Text GLabel 7500 4200 2    50   Input ~ 0
 SPI-CLK
-Text GLabel 7500 4200 2    50   Input ~ 0
-SPI-SDO
+Text GLabel 3900 3700 2    50   Input ~ 0
+SPI-MOSI
 $EndSCHEMATC

Commit message: add footprints, clear board
Other:
- moved on the sheet: DSUB2, T1, T2, U1
Changed lines of the file:
@@
 EELAYER 30 0
 EELAYER END
-$Descr A4 11693 8268
+$Descr A4 8268 11693 portrait
 encoding utf-8
 Sheet 1 1
@@
 Comment4 ""
 $EndDescr
-Text GLabel 3900 3200 2    50   Input ~ 0
+Text GLabel 4100 3250 2    50   Input ~ 0
 1Wire
-Text GLabel 3900 3600 2    50   Input ~ 0
+Text GLabel 4100 3650 2    50   Input ~ 0
 DHT22
 $Comp
 L Connector:DB9_Female_MountingHoles DSUB2
 U 1 1 5F245498
-P 3600 3400
-F 0 "DSUB2" H 3780 3309 50  0000 L CNN
-F 1 "DB9_Female" H 3780 3400 50  0000 L CNN
-F 2 "Connector_Dsub:DSUB-9_Female_Horizontal_P2.77x2.84mm_EdgePinOffset4.94mm_Housed_MountingHolesOffset7.48mm" H 3600 3400 50  0001 C CNN
-F 3 " ~" H 3600 3400 50  0001 C CNN
-	1    3600 3400
+P 3800 3450
+F 0 "DSUB2" H 3980 3359 50  0000 L CNN
+F 1 "DB9_Female" H 3980 3450 50  0000 L CNN
+F 2 "Connector_Dsub:DSUB-9_Female_Horizontal_P2.77x2.84mm_EdgePinOffset4.94mm_Housed_MountingHolesOffset7.48mm" H 3800 3450 50  0001 C CNN
+F 3 " ~" H 3800 3450 50  0001 C CNN
+	1    3800 3450
 	-1   0    0    1
 $EndComp
 Wire Wire Line
-	3600 2450 3600 2800
-Wire Wire Line
-	3900 2450 3600 2450
-Wire Wire Line
-	3900 2650 3900 2450
+	3800 2500 3800 2850
+Wire Wire Line
+	4100 2500 3800 2500
+Wire Wire Line
+	4100 2700 4100 2500
 $Comp
 L power:GND #PWR0121
 U 1 1 5F764AC1
-P 3900 2650
-F 0 "#PWR0121" H 3900 2400 50  0001 C CNN
-F 1 "GND" H 3905 2477 50  0000 C CNN
-F 2 "" H 3900 2650 50  0001 C CNN
-F 3 "" H 3900 2650 50  0001 C CNN
-	1    3900 2650
+P 4100 2700
+F 0 "#PWR0121" H 4100 2450 50  0001 C CNN
+F 1 "GND" H 4105 2527 50  0000 C CNN
+F 2 "" H 4100 2700 50  0001 C CNN
+F 3 "" H 4100 2700 50  0001 C CNN
+	1    4100 2700
 	1    0    0    -1
 $EndComp
@@
 L power:+5V #PWR0125
 U 1 1 5F25599A
-P 4100 2800
-F 0 "#PWR0125" H 4100 2650 50  0001 C CNN
-F 1 "+5V" H 4115 2973 50  0000 C CNN
-F 2 "" H 4100 2800 50  0001 C CNN
-F 3 "" H 4100 2800 50  0001 C CNN
-	1    4100 2800
-	1    0    0    -1
-$EndComp
-Wire Wire Line
-	4100 3000 4100 2800
-Wire Wire Line
-	3900 3000 4100 3000
-Wire Wire Line
-	4100 4000 4100 3800
+P 4300 2850
+F 0 "#PWR0125" H 4300 2700 50  0001 C CNN
+F 1 "+5V" H 4315 3023 50  0000 C CNN
+F 2 "" H 4300 2850 50  0001 C CNN
+F 3 "" H 4300 2850 50  0001 C CNN
+	1    4300 2850
+	1    0    0    -1
+$EndComp
+Wire Wire Line
+	4300 3050 4300 2850
+Wire Wire Line
+	4100 3050 4300 3050
+Wire Wire Line
+	4300 4050 4300 3850
 $Comp
 L power:GND #PWR0116
 U 1 1 5F75D03D
-P 4100 4000
-F 0 "#PWR0116" H 4100 3750 50  0001 C CNN
-F 1 "GND" H 4105 3827 50  0000 C CNN
-F 2 "" H 4100 4000 50  0001 C CNN
-F 3 "" H 4100 4000 50  0001 C CNN
-	1    4100 4000
-	1    0    0    -1
-$EndComp
-Wire Wire Line
-	3900 3800 4100 3800
+P 4300 4050
+F 0 "#PWR0116" H 4300 3800 50  0001 C CNN
+F 1 "GND" H 4305 3877 50  0000 C CNN
+F 2 "" H 4300 4050 50  0001 C CNN
+F 3 "" H 4300 4050 50  0001 C CNN
+	1    4300 4050
+	1    0    0    -1
+$EndComp
+Wire Wire Line
+	4100 3850 4300 3850
 $Comp
 L power:+5V #PWR0101
 U 1 1 5EA2BC90
-P 9000 3750
-F 0 "#PWR0101" H 9000 3600 50  0001 C CNN
-F 1 "+5V" H 9015 3923 50  0000 C CNN
-F 2 "" H 9000 3750 50  0001 C CNN
-F 3 "" H 9000 3750 50  0001 C CNN
-	1    9000 3750
+P 5000 7150
+F 0 "#PWR0101" H 5000 7000 50  0001 C CNN
+F 1 "+5V" H 5015 7323 50  0000 C CNN
+F 2 "" H 5000 7150 50  0001 C CNN
+F 3 "" H 5000 7150 50  0001 C CNN
+	1    5000 7150
 	-1   0    0    -1
 $EndComp
@@
 L power:GND #PWR0102
 U 1 1 5EA2BC96
-P 9000 4350
-F 0 "#PWR0102" H 9000 4100 50  0001 C CNN
-F 1 "GND" H 9005 4177 50  0000 C CNN
-F 2 "" H 9000 4350 50  0001 C CNN
-F 3 "" H 9000 4350 50  0001 C CNN
-	1    9000 4350
+P 5000 7750
+F 0 "#PWR0102" H 5000 7500 50  0001 C CNN
+F 1 "GND" H 5005 7577 50  0000 C CNN
+F 2 "" H 5000 7750 50  0001 C CNN
+F 3 "" H 5000 7750 50  0001 C CNN
+	1    5000 7750
 	-1   0    0    -1
 $EndComp
@@
 L Sensor:DHT11 U1
 U 1 1 5EA2BC9C
-P 9000 4050
-F 0 "U1" H 8700 4100 50  0000 R CNN
-F 1 "DHT22" H 8700 4000 50  0000 R CNN
-F 2 "Sensor:Aosong_DHT11_5.5x12.0_P2.54mm" H 9000 3650 50  0001 C CNN
-F 3 "https://www.sparkfun.com/datasheets/Sensors/Temperature/DHT22.pdf" H 9150 4300 50  0001 C CNN
-	1    9000 4050
+P 5000 7450
+F 0 "U1" H 4700 7500 50  0000 R CNN
+F 1 "DHT22" H 4700 7400 50  0000 R CNN
+F 2 "Sensor:Aosong_DHT11_5.5x12.0_P2.54mm" H 5000 7050 50  0001 C CNN
+F 3 "https://www.sparkfun.com/datasheets/Sensors/Temperature/DHT22.pdf" H 5150 7700 50  0001 C CNN
+	1    5000 7450
 	-1   0    0    -1
 $EndComp
@@
 L power:GND #PWR0104
 U 1 1 5EA2BCA2
-P 9000 2950
-F 0 "#PWR0104" H 9000 2700 50  0001 C CNN
-F 1 "GND" H 9005 2777 50  0000 C CNN
-F 2 "" H 9000 2950 50  0001 C CNN
-F 3 "" H 9000 2950 50  0001 C CNN
-	1    9000 2950
+P 5000 6350
+F 0 "#PWR0104" H 5000 6100 50  0001 C CNN
+F 1 "GND" H 5005 6177 50  0000 C CNN
+F 2 "" H 5000 6350 50  0001 C CNN
+F 3 "" H 5000 6350 50  0001 C CNN
+	1    5000 6350
 	-1   0    0    -1
 $EndComp
@@
 L power:+5V #PWR0105
 U 1 1 5EA2BCA8
-P 9000 2350
-F 0 "#PWR0105" H 9000 2200 50  0001 C CNN
-F 1 "+5V" H 9015 2523 50  0000 C CNN
-F 2 "" H 9000 2350 50  0001 C CNN
-F 3 "" H 9000 2350 50  0001 C CNN
-	1    9000 2350
+P 5000 5750
+F 0 "#PWR0105" H 5000 5600 50  0001 C CNN
+F 1 "+5V" H 5015 5923 50  0000 C CNN
+F 2 "" H 5000 5750 50  0001 C CNN
+F 3 "" H 5000 5750 50  0001 C CNN
+	1    5000 5750
 	-1   0    0    -1
 $EndComp
@@
 L power:+5V #PWR0106
 U 1 1 5EA2BCAE
-P 7100 2350
-F 0 "#PWR0106" H 7100 2200 50  0001 C CNN
-F 1 "+5V" H 7115 2523 50  0000 C CNN
-F 2 "" H 7100 2350 50  0001 C CNN
-F 3 "" H 7100 2350 50  0001 C CNN
-	1    7100 2350
+P 3100 5750
+F 0 "#PWR0106" H 3100 5600 50  0001 C CNN
+F 1 "+5V" H 3115 5923 50  0000 C CNN
+F 2 "" H 3100 5750 50  0001 C CNN
+F 3 "" H 3100 5750 50  0001 C CNN
+	1    3100 5750
 	-1   0    0    -1
 $EndComp
@@
 L power:GND #PWR0107
 U 1 1 5EA2BCB4
-P 7100 2950
-F 0 "#PWR0107" H 7100 2700 50  0001 C CNN
-F 1 "GND" H 7105 2777 50  0000 C CNN
-F 2 "" H 7100 2950 50  0001 C CNN
-F 3 "" H 7100 2950 50  0001 C CNN
-	1    7100 2950
+P 3100 6350
+F 0 "#PWR0107" H 3100 6100 50  0001 C CNN
+F 1 "GND" H 3105 6177 50  0000 C CNN
+F 2 "" H 3100 6350 50  0001 C CNN
+F 3 "" H 3100 6350 50  0001 C CNN
+	1    3100 6350
 	-1   0    0    -1
 $EndComp
@@
 L Sensor_Temperature:DS18B20 T1
 U 1 1 5EA2BCBA
-P 7100 2650
-F 0 "T1" H 6800 2700 50  0000 R CNN
-F 1 "DS18B20" H 6800 2600 50  0000 R CNN
-F 2 "Package_TO_SOT_THT:TO-92_Inline_Wide" H 6100 2400 50  0001 C CNN
-F 3 "http://datasheets.maximintegrated.com/en/ds/DS18B20.pdf" H 6950 2900 50  0001 C CNN
-	1    7100 2650
+P 3100 6050
+F 0 "T1" H 2800 6100 50  0000 R CNN
+F 1 "DS18B20" H 2800 6000 50  0000 R CNN
+F 2 "Package_TO_SOT_THT:TO-92_Inline_Wide" H 2100 5800 50  0001 C CNN
+F 3 "http://datasheets.maximintegrated.com/en/ds/DS18B20.pdf" H 2950 6300 50  0001 C CNN
+	1    3100 6050
 	-1   0    0    -1
 $EndComp
@@
 L Sensor_Temperature:DS18B20 T2
 U 1 1 5EA2BCC0
-P 9000 2650
-F 0 "T2" H 8700 2700 50  0000 R CNN
-F 1 "DS18B20" H 8700 2600 50  0000 R CNN
-F 2 "Package_TO_SOT_THT:TO-92_Inline_Wide" H 8000 2400 50  0001 C CNN
-F 3 "http://datasheets.maximintegrated.com/en/ds/DS18B20.pdf" H 8850 2900 50  0001 C CNN
-	1    9000 2650
-	-1   0    0    -1
-$EndComp
-Text GLabel 8700 2650 0    50   Input ~ 0
+P 5000 6050
+F 0 "T2" H 4700 6100 50  0000 R CNN
+F 1 "DS18B20" H 4700 6000 50  0000 R CNN
+F 2 "Package_TO_SOT_THT:TO-92_Inline_Wide" H 4000 5800 50  0001 C CNN
+F 3 "http://datasheets.maximintegrated.com/en/ds/DS18B20.pdf" H 4850 6300 50  0001 C CNN
+	1    5000 6050
+	-1   0    0    -1
+$EndComp
+Text GLabel 4700 6050 0    50   Input ~ 0
 1Wire
-Text GLabel 6800 2650 0    50   Input ~ 0
+Text GLabel 2800 6050 0    50   Input ~ 0
 1Wire
-Text GLabel 8700 4050 0    50   Input ~ 0
+Text GLabel 4700 7450 0    50   Input ~ 0
 DHT22
 $Comp
 L Sensor_Pressure:MS5607-02BA U9
 U 1 1 5EA6EE10
-P 7100 4100
-F 0 "U9" H 7430 4146 50  0000 L CNN
-F 1 "SSCDRNN015PASA5" H 7430 4055 50  0000 L CNN
-F 2 "Package_DIP:DIP-8_W8.89mm_SMDSocket_LongPads" H 7100 4100 50  0001 C CNN
-F 3 "https://sensing.honeywell.com/index.php?ci_id=151134" H 7100 4100 50  0001 C CNN
-	1    7100 4100
+P 3100 7500
+F 0 "U9" H 3430 7546 50  0000 L CNN
+F 1 "SSCDRNN015PASA5" H 3430 7455 50  0000 L CNN
+F 2 "Package_DIP:DIP-8_W8.89mm_SMDSocket_LongPads" H 3100 7500 50  0001 C CNN
+F 3 "https://sensing.honeywell.com/index.php?ci_id=151134" H 3100 7500 50  0001 C CNN
+	1    3100 7500
 	-1   0    0    -1
 $EndComp
@@
 L power:GND #PWR0122
 U 1 1 5EA710CD
-P 7100 4500
-F 0 "#PWR0122" H 7100 4250 50  0001 C CNN
-F 1 "GND" H 7105 4327 50  0000 C CNN
-F 2 "" H 7100 4500 50  0001 C CNN
-F 3 "" H 7100 4500 50  0001 C CNN
-	1    7100 4500
-	1    0    0    -1
-$EndComp
-Text GLabel 7500 4300 2    50   Input ~ 0
+P 3100 7900
+F 0 "#PWR0122" H 3100 7650 50  0001 C CNN
+F 1 "GND" H 3105 7727 50  0000 C CNN
+F 2 "" H 3100 7900 50  0001 C CNN
+F 3 "" H 3100 7900 50  0001 C CNN
+	1    3100 7900
+	1    0    0    -1
+$EndComp
+Text GLabel 3500 7700 2    50   Input ~ 0
 SPI-SS-Pressure
 $Comp
@@
 	1    0    0    -1
 $EndComp
-Text GLabel 3900 3400 2    50   Input ~ 0
+Text GLabel 4100 3450 2    50   Input ~ 0
 SPI-MISO
-Text GLabel 3900 3500 2    50   Input ~ 0
+Text GLabel 4100 3550 2    50   Input ~ 0
 SPI-SS-Pressure
 $Comp
 L power:+5V #PWR0108
 U 1 1 5EAA384C
-P 7100 3700
-F 0 "#PWR0108" H 7100 3550 50  0001 C CNN
-F 1 "+5V" H 7115 3873 50  0000 C CNN
-F 2 "" H 7100 3700 50  0001 C CNN
-F 3 "" H 7100 3700 50  0001 C CNN
-	1    7100 3700
-	-1   0    0    -1
-$EndComp
-Text GLabel 3900 3300 2    50   Input ~ 0
+P 3100 7100
+F 0 "#PWR0108" H 3100 6950 50  0001 C CNN
+F 1 "+5V" H 3115 7273 50  0000 C CNN
+F 2 "" H 3100 7100 50  0001 C CNN
+F 3 "" H 3100 7100 50  0001 C CNN
+	1    3100 7100
+	-1   0    0    -1
+$EndComp
+Text GLabel 4100 3350 2    50   Input ~ 0
 SPI-CLK
-Text GLabel 7500 4000 2    50   Input ~ 0
+Text GLabel 3500 7400 2    50   Input ~ 0
 SPI-MISO
-Text GLabel 7500 4200 2    50   Input ~ 0
+Text GLabel 3500 7600 2    50   Input ~ 0
 SPI-CLK
-Text GLabel 3900 3700 2    50   Input ~ 0
+Text GLabel 4100 3750 2    50   Input ~ 0
 SPI-MOSI
 $EndSCHEMATC

Commit message: fix pressure sensor footprint
Parts:
- removed U9: SSCDRNN015PASA5, Package_DIP:DIP-8_W8.89mm_SMDSocket_LongPads, symbol Sensor_Pressure:MS5607-02BA
- added U?: SSCDRNN015PASA5, Package_DIP:DIP-8_W8.89mm_SMDSocket_LongPads, symbol sscdrnn015pasa5:SSCDRNN015PASA5
Changed lines of the file:
@@
 DHT22
-$Comp
-L Sensor_Pressure:MS5607-02BA U9
-U 1 1 5EA6EE10
-P 3100 7500
-F 0 "U9" H 3430 7546 50  0000 L CNN
-F 1 "SSCDRNN015PASA5" H 3430 7455 50  0000 L CNN
-F 2 "Package_DIP:DIP-8_W8.89mm_SMDSocket_LongPads" H 3100 7500 50  0001 C CNN
-F 3 "https://sensing.honeywell.com/index.php?ci_id=151134" H 3100 7500 50  0001 C CNN
-	1    3100 7500
-	-1   0    0    -1
-$EndComp
 $Comp
 L power:GND #PWR0122
 U 1 1 5EA710CD
-P 3100 7900
-F 0 "#PWR0122" H 3100 7650 50  0001 C CNN
-F 1 "GND" H 3105 7727 50  0000 C CNN
-F 2 "" H 3100 7900 50  0001 C CNN
-F 3 "" H 3100 7900 50  0001 C CNN
-	1    3100 7900
+P 3100 7800
+F 0 "#PWR0122" H 3100 7550 50  0001 C CNN
+F 1 "GND" H 3105 7627 50  0000 C CNN
+F 2 "" H 3100 7800 50  0001 C CNN
+F 3 "" H 3100 7800 50  0001 C CNN
+	1    3100 7800
 	1    0    0    -1
 $EndComp
-Text GLabel 3500 7700 2    50   Input ~ 0
+Text GLabel 3500 7350 2    50   Input ~ 0
 SPI-SS-Pressure
 $Comp
@@
 L power:+5V #PWR0108
 U 1 1 5EAA384C
-P 3100 7100
-F 0 "#PWR0108" H 3100 6950 50  0001 C CNN
-F 1 "+5V" H 3115 7273 50  0000 C CNN
-F 2 "" H 3100 7100 50  0001 C CNN
-F 3 "" H 3100 7100 50  0001 C CNN
-	1    3100 7100
+P 3100 7050
+F 0 "#PWR0108" H 3100 6900 50  0001 C CNN
+F 1 "+5V" H 3115 7223 50  0000 C CNN
+F 2 "" H 3100 7050 50  0001 C CNN
+F 3 "" H 3100 7050 50  0001 C CNN
+	1    3100 7050
 	-1   0    0    -1
 $EndComp
 Text GLabel 4100 3350 2    50   Input ~ 0
 SPI-CLK
-Text GLabel 3500 7400 2    50   Input ~ 0
+Text GLabel 3500 7550 2    50   Input ~ 0
 SPI-MISO
-Text GLabel 3500 7600 2    50   Input ~ 0
+Text GLabel 3500 7450 2    50   Input ~ 0
 SPI-CLK
 Text GLabel 4100 3750 2    50   Input ~ 0
 SPI-MOSI
+$Comp
+L sscdrnn015pasa5:SSCDRNN015PASA5 U?
+U 1 1 5EA36ED1
+P 3100 8000
+F 0 "U?" H 2771 8621 50  0000 R CNN
+F 1 "SSCDRNN015PASA5" H 2771 8530 50  0000 R CNN
+F 2 "Package_DIP:DIP-8_W8.89mm_SMDSocket_LongPads" H 3100 8000 50  0001 C CNN
+F 3 "https://sensing.honeywell.com/index.php?ci_id=151134" H 3100 8000 50  0001 C CNN
+	1    3100 8000
+	1    0    0    -1
+$EndComp
 $EndSCHEMATC

Commit message: add db9 models, and update footprints
Parts:
- DSUB2: value DB9_Female -> DB9_Male; footprint Connector_Dsub:DSUB-9_Female_Horizontal_P2.77x2.84mm_EdgePinOffset4.94mm_Housed_MountingHolesOffset7.48mm -> Connector_Dsub:DSUB-9_Male_Horizontal_P2.77x2.84mm_EdgePinOffset7.70mm_Housed_MountingHolesOffset9.12mm; symbol Connector:DB9_Female_MountingHoles -> Connector:DB9_Male_MountingHoles
- gave numbers to parts that had none: 1
Connections:
- net +5V: now also DSUB2.1; no longer DSUB2.5
- net 1Wire: now also DSUB2.2; no longer DSUB2.4
- net DHT22: now also DSUB2.4; no longer DSUB2.2
- net GND: now also DSUB2.5; no longer DSUB2.1
- net SPI-CLK: now also DSUB2.7; no longer DSUB2.8
- net SPI-MOSI: now also DSUB2.9; no longer DSUB2.6
- net SPI-SS-Pressure: now also DSUB2.8; no longer DSUB2.7
Changed lines of the file:
@@
 DHT22
 $Comp
-L Connector:DB9_Female_MountingHoles DSUB2
+L Connector:DB9_Male_MountingHoles DSUB2
 U 1 1 5F245498
 P 3800 3450
 F 0 "DSUB2" H 3980 3359 50  0000 L CNN
-F 1 "DB9_Female" H 3980 3450 50  0000 L CNN
-F 2 "Connector_Dsub:DSUB-9_Female_Horizontal_P2.77x2.84mm_EdgePinOffset4.94mm_Housed_MountingHolesOffset7.48mm" H 3800 3450 50  0001 C CNN
+F 1 "DB9_Male" H 3980 3450 50  0000 L CNN
+F 2 "Connector_Dsub:DSUB-9_Male_Horizontal_P2.77x2.84mm_EdgePinOffset7.70mm_Housed_MountingHolesOffset9.12mm" H 3800 3450 50  0001 C CNN
 F 3 " ~" H 3800 3450 50  0001 C CNN
 	1    3800 3450
@@
 SPI-MOSI
 $Comp
-L sscdrnn015pasa5:SSCDRNN015PASA5 U?
+L sscdrnn015pasa5:SSCDRNN015PASA5 U2
 U 1 1 5EA36ED1
 P 3100 8000
-F 0 "U?" H 2771 8621 50  0000 R CNN
+F 0 "U2" H 2771 8621 50  0000 R CNN
 F 1 "SSCDRNN015PASA5" H 2771 8530 50  0000 R CNN
 F 2 "Package_DIP:DIP-8_W8.89mm_SMDSocket_LongPads" H 3100 8000 50  0001 C CNN

Commit message: WIP sensor PCB
Parts:
- removed DSUB2: DB9_Male, Connector_Dsub:DSUB-9_Male_Horizontal_P2.77x2.84mm_EdgePinOffset7.70mm_Housed_MountingHolesOffset9.12mm, symbol Connector:DB9_Male_MountingHoles
- removed T1, T2: DS18B20, Package_TO_SOT_THT:TO-92_Inline_Wide, symbol Sensor_Temperature:DS18B20
- added D1, D10, D11, D12, D13, D14, D15, D16, D2, D3, D4, D5, D6, D7, D8, D9: LED, LED_SMD:LED_0805_2012Metric_Pad1.15x1.40mm_HandSolder, symbol Device:LED
- added J1: Conn_01x08_Female, Stardust:691382040008, symbol Connector:Conn_01x08_Female
- added R1: R10k, Resistor_SMD:R_0603_1608Metric_Pad0.98x0.95mm_HandSolder, symbol Device:R
- added R10, R11, R12, R13, R14, R15, R16, R17, R2, R3, R4, R5, R6, R7, R8, R9: R330, Resistor_SMD:R_0603_1608Metric, symbol Device:R
- added U3: TCA9555DBR, Package_SO:SSOP-24_5.3x8.2mm_P0.65mm, symbol Interface_Expansion:TCA9555DBR
- U1: footprint Sensor:Aosong_DHT11_5.5x12.0_P2.54mm -> Stardust:DHT22_15.0x25.0_P2.54mm_Horizontal
Connections:
- net +5V: now also J1.8 (Pin_8), R1.1, U3.24 (VCC)
- net DHT22: now also J1.2 (Pin_2)
- net GND: now also D1.1 (K), D10.1 (K), D11.1 (K), D12.1 (K), D13.1 (K), D14.1 (K), D15.1 (K), D16.1 (K), D2.1 (K), D3.1 (K), D4.1 (K), D5.1 (K), D6.1 (K), D7.1 (K), D8.1 (K), D9.1 (K), J1.1 (Pin_1), U3.12 (GND), U3.2 (A1), U3.21 (A0), U3.3 (A2)
- net SPI-CLK: now also J1.5 (Pin_5)
- net SPI-MISO: now also J1.6 (Pin_6)
- net SPI-SS-Pressure: now also J1.7 (Pin_7)
- new net: D9.2 (A), R3.1
- new net: D2.2 (A), R4.1
- new net: R4.2, U3.6 (P02)
- new net: D10.2 (A), R5.1
- new net: R5.2, U3.7 (P03)
- new net: D3.2 (A), R6.1
- new net: R6.2, U3.8 (P04)
- new net: D11.2 (A), R7.1
- new net: R7.2, U3.9 (P05)
- new net: D4.2 (A), R8.1
- new net: R8.2, U3.10 (P06)
- new net: D12.2 (A), R9.1
- new net: R9.2, U3.11 (P07)
- new net: D5.2 (A), R10.1
- new net: R10.2, U3.13 (P10)
- new net: D13.2 (A), R11.1
- new net: R11.2, U3.14 (P11)
- new net: D6.2 (A), R12.1
- new net: R12.2, U3.15 (P12)
- new net: D14.2 (A), R13.1
- new net: R13.2, U3.16 (P13)
- new net: D7.2 (A), R14.1
- new net: R14.2, U3.17 (P14)
- new net: D15.2 (A), R15.1
- new net: R15.2, U3.18 (P15)
- new net: D8.2 (A), R16.1
- new net: R16.2, U3.19 (P16)
- new net: D16.2 (A), R17.1
- new net: R17.2, U3.20 (P17)
- new net: R1.2, U3.1 (~INT)
- new net: R2.2, U3.4 (P00)
- new net: R3.2, U3.5 (P01)
- new net: D1.2 (A), R2.1
- new net SCL: J1.4 (Pin_4), U3.22 (SCL)
- new net SDA: J1.3 (Pin_3), U3.23 (SDA)
Other:
- moved on the sheet: U1, U2

Commit message: WIP sensor PCB - delete files
Parts:
- U2: symbol sscdrnn015pasa5:SSCDRNN015PASA5 -> Stardust:SSCDRNN015PASA5
Changed lines of the file:
@@
 SPI-CLK
 $Comp
-L sscdrnn015pasa5:SSCDRNN015PASA5 U2
+L Stardust:SSCDRNN015PASA5 U2
 U 1 1 5EA36ED1
 P 2950 4650

Commit message: WIP
Changed lines of the file:
@@
 U 1 1 601916EE
 P 3700 6900
-F 0 "U3" H 3700 8181 50  0000 C CNN
+F 0 "U3" H 3950 7950 50  0000 C CNN
 F 1 "TCA9555DBR" H 3950 7850 50  0000 C CNN
 F 2 "Package_SO:SSOP-24_5.3x8.2mm_P0.65mm" H 4750 5900 50  0001 C CNN
